File: imu_rc_car/pcb/imu_rc_car.kicad_sch (KiCad schematic)
At the start: 0 parts

Commit message: commit #15
started car board development
added encoders schematic
added prox sensors schematic
refactored battery send src code
added future development code
Parts:
- added U1: ESP32-S3-DevKitC, PCM_Espressif:ESP32-S3-DevKitC, symbol PCM_Espressif:ESP32-S3-DevKitC
Connections:
- new net: U1.1 (3V3), U1.2 (3V3)
- new net: U1.22 (GND), U1.23 (GND), U1.24 (GND), U1.44 (GND)
Other:
- added sheet Encoders (encoders.kicad_sch)
- added sheet Prox Sensors (prox_sensors.kicad_sch)
Changed lines of the file:
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@@
 		(company "ESTG-IPL")
+	)
+	(symbol
+		(lib_id "PCM_Espressif:ESP32-S3-DevKitC")
+		(at 209.55 132.08 0)
+		(unit 1)
+		(exclude_from_sim no)
+		(in_bom yes)
+		(on_board yes)
+		(dnp no)
+		(fields_autoplaced yes)
+		(property "Reference" "U1"
+			(at 211.7441 177.8 0)
+			(effects
+				(font
+					(size 1.27 1.27)
+				)
+				(justify left)
+			)
+		)
+		(property "Value" "ESP32-S3-DevKitC"
+			(at 211.7441 180.34 0)
+			(effects
+				(font
+					(size 1.27 1.27)
+				)
+				(justify left)
+			)
+		)
+		(property "Footprint" "PCM_Espressif:ESP32-S3-DevKitC"
+			(at 209.55 189.23 0)
+			(effects
+				(font
+					(size 1.27 1.27)
+				)
+				(hide yes)
+			)
+		)
+		(property "Datasheet" ""
+			(at 149.86 134.62 0)
+			(effects
+				(font
+					(size 1.27 1.27)
+				)
+				(hide yes)
+			)
+		)
+		(property "Description" "ESP32-S3-DevKitC"
+			(at 209.55 132.08 0)
+			(effects
+				(font
+					(size 1.27 1.27)
+				)
+				(hide yes)
+			)
+		)
+		(pin "9"
+		)
+		(pin "40"
+		)
+		(pin "2"
+		)
+		(pin "3"
+		)
+		(pin "29"
+		)
+		(pin "43"
+		)
+		(pin "34"
+		)
+		(pin "15"
+		)
+		(pin "18"
+		)
+		(pin "25"
+		)
+		(pin "39"
+		)
+		(pin "41"
+		)
+		(pin "42"
+		)
+		(pin "17"
+		)
+		(pin "27"
+		)
+		(pin "28"
+		)
+		(pin "16"
+		)
+		(pin "13"
+		)
+		(pin "4"
+		)
+		(pin "11"
+		)
+		(pin "23"
+		)
+		(pin "1"
+		)
+		(pin "14"
+		)
+		(pin "22"
+		)
+		(pin "10"
+		)
+		(pin "30"
+		)
+		(pin "31"
+		)
+		(pin "32"
+		)
+		(pin "20"
+		)
+		(pin "24"
+		)
+		(pin "33"
+		)
+		(pin "12"
+		)
+		(pin "38"
+		)
+		(pin "5"
+		)
+		(pin "6"
+		)
+		(pin "44"
+		)
+		(pin "21"
+		)
+		(pin "7"
+		)
+		(pin "8"
+		)
+		(pin "19"
+		)
+		(pin "26"
+		)
+		(pin "35"
+		)
+		(pin "36"
+		)
+		(pin "37"
+		)
+		(instances
+			(project ""
+				(path "/34ec7d21-7026-4230-8659-e414bc456131"
+					(reference "U1")
+					(unit 1)
+				)
+			)
+		)
+	)
+	(sheet
+		(at 238.76 260.35)
+		(size 27.94 13.97)
+		(fields_autoplaced yes)
+		(stroke
+			(width 0.1524)
+			(type solid)
+		)
+		(fill
+			(color 0 0 0 0.0000)
+		)
+		(property "Sheetname" "Prox Sensors"
+			(at 238.76 259.6384 0)
+			(effects
+				(font
+					(size 1.27 1.27)
+				)
+				(justify left bottom)
+			)
+		)
+		(property "Sheetfile" "prox_sensors.kicad_sch"
+			(at 238.76 274.9046 0)
+			(effects
+				(font
+					(size 1.27 1.27)
+				)
+				(justify left top)
+			)
+		)
+		(instances
+			(project "imu_rc_car"
+				(path "/34ec7d21-7026-4230-8659-e414bc456131"
+					(page "3")
+				)
+			)
+		)
+	)
+	(sheet
+		(at 267.97 260.35)
+		(size 27.94 13.97)
+		(fields_autoplaced yes)
+		(stroke
+			(width 0.1524)
+			(type solid)
+		)
+		(fill
+			(color 0 0 0 0.0000)
+		)
+		(property "Sheetname" "Encoders"
+			(at 267.97 259.6384 0)
+			(effects
+				(font
+					(size 1.27 1.27)
+				)
+				(justify left bottom)
+			)
+		)
+		(property "Sheetfile" "encoders.kicad_sch"
+			(at 267.97 274.9046 0)
+			(effects
+				(font
+					(size 1.27 1.27)
+				)
+				(justify left top)
+			)
+		)
+		(instances
+			(project "imu_rc_car"
+				(path "/34ec7d21-7026-4230-8659-e414bc456131"
+					(page "2")
+				)
+			)
+		)
 	)
 	(sheet_instances

Commit message: commit #18
added text in encoder board
added pcb layout for car
started car schematic
Parts:
- added C1, C2, C3, C4, C5, C6: 10uF, Capacitor_SMD:C_1206_3216Metric_Pad1.33x1.80mm_HandSolder, symbol Device:C
- added J1: Encoder FS, Connector_JST:JST_PH_S4B-PH-K_1x04_P2.00mm_Horizontal, symbol Connector:Conn_01x04_Socket
- added J2: Encoder BS, Connector_JST:JST_PH_S4B-PH-K_1x04_P2.00mm_Horizontal, symbol Connector:Conn_01x04_Socket
- added J3: Prox Sensor FS, Connector:FanPinHeader_1x03_P2.54mm_Vertical, symbol Connector:Conn_01x03_Socket
- added J4: Prox Sensor RS, Connector:FanPinHeader_1x03_P2.54mm_Vertical, symbol Connector:Conn_01x03_Socket
- added J5: Prox Sensor LS, Connector:FanPinHeader_1x03_P2.54mm_Vertical, symbol Connector:Conn_01x03_Socket
- added J6: Prox Sensor BS, Connector:FanPinHeader_1x03_P2.54mm_Vertical, symbol Connector:Conn_01x03_Socket
Connections:
- net +3V3: now reaches U1.1 (3V3), U1.2 (3V3)
- net +3V3: now also C1.1, C2.1, C3.1, C4.1, C5.1, C6.1, J1.4 (Pin_4), J2.4 (Pin_4), J3.3 (Pin_3), J4.3 (Pin_3), J5.3 (Pin_3), J6.3 (Pin_3)
- net GND: now reaches U1.22 (GND), U1.23 (GND), U1.24 (GND), U1.44 (GND)
- net GND: now also C1.2, C2.2, C3.2, C4.2, C5.2, C6.2, J1.3 (Pin_3), J2.3 (Pin_3), J3.2 (Pin_2), J4.2 (Pin_2), J5.2 (Pin_2), J6.2 (Pin_2)
- new net ENC1: J1.2 (Pin_2)
- new net ENC2: J1.1 (Pin_1)
- new net ENC3: J2.2 (Pin_2)
- new net ENC4: J2.1 (Pin_1)
- new net PRX_BS: J6.1 (Pin_1)
- new net PRX_FS: J3.1 (Pin_1)
- new net PRX_LS: J5.1 (Pin_1)
- new net PRX_RS: J4.1 (Pin_1)
Other:
- removed sheet Encoders
- removed sheet Prox Sensors
