File: imu_rc_car/pcb/imu_rc_car_prox_sensors/imu_rc_car_prox_sensors.kicad_sch (KiCad schematic)
At the start: 12 parts, among them J1 Conn_01x05_Socket

Commit message: commit #27
revision for hand unit complete (board is ready)
board for proximity sensors in series
minor revision in encoder board
progressing work in car board
added essential libraries support for 3D components
Other:
- moved on the sheet: C1, C2, D1, J1, R1

Commit message: commit #32
costs table 4
first revision of imu rc car pcb
imu rc encoders final version v1.0.0 (ordered)
imu rc prox sensors final version v1.0.0 (ordered)
minor resistors tolerance changes in hand unit
Parts:
- D2: value IR204A -> IR333C-A
- D3: value AA -> PD333-3B
- R3: value 43 (1%) -> 1800 (1%)
- R4: value 4k02 (1%) -> 150k (1%)
Other:
- moved on the sheet: C3, C4, D2, R3, R4
