File: imu_rc_hand_unit/pcb/v1.1.0/imu_rc_hand_unit.kicad_pcb (KiCad board)
At the start: 2 copper layers, 35 x 50 mm, 80 parts, among them J1 USB_C_Receptacle_USB2.0_16P, J2 JST SH1.0, Q1 IRLML6344TRPBF, Q2 IRLML6344TRPBF, Q3 DMP3160L-7, Q4 IRLML6344TRPBF, Q5 DMP3160L-7, Q6 BSS138, Q7 BC817-25, Q8 BC817-25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

Commit message: commit #36
added project report
few changes in imu rc car chassis for 3d printing
fixed some imu rc car pin outputs
major folder hierarchy refactor in pcb hand unit

imu rc hand unit v1.2.0:
changed footprint of MCP73831 to DFN-8
added 3V3 to VIO pin in CP2102N

new imu rc hand unit v2.0.0:
Changed to MCP73871
Removed BQ297
Removed a few components
only schematic is done
Parts:
- C12, C14, C15, C17, C18, C19, C20, C8: value 100nF/50V(10%) -> 100nF/50V
- C13, C2, C4: value 1uF/16V(10%) -> 1uF/16V
- C5: value 0.1uF/16V -> 100nF/16V
- D1, D2: value LESD5D5.0CT1G -> ESD5B5V0WT
- R1, R2: value 5k1 (1%) -> 5k1
- R13: value 3k (1%) -> 3k
- R14: value 11k (1%) -> 11k
- R20, R21, R9: value 2k2 (1%) -> 2k2
- R31: value 150 -> 330
- R32: value 33 -> 68
- R33: value 10 -> 68
Changed lines of the file:
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@@
 			)
 		)
-		(property "Value" "10"
+		(property "Value" "68"
 			(at 0 1.65 90)
 			(layer "F.Fab")
@@
 			)
 		)
-		(property "Value" "100nF/50V(10%)"
+		(property "Value" "100nF/50V"
 			(at 0 1.68 0)
 			(layer "F.Fab")
@@
 			)
 		)
-		(property "Value" "100nF/50V(10%)"
+		(property "Value" "100nF/50V"
 			(at 0 1.68 0)
 			(layer "F.Fab")
@@
 			)
 		)
-		(property "Value" "100nF/50V(10%)"
+		(property "Value" "100nF/50V"
 			(at 0 1.68 0)
 			(layer "F.Fab")
@@
 			)
 		)
-		(property "Value" "33"
+		(property "Value" "68"
 			(at 0 1.65 0)
 			(layer "F.Fab")
@@
 			)
 		)
-		(property "Value" "150"
+		(property "Value" "330"
 			(at 0 1.65 0)
 			(layer "F.Fab")
@@
 			)
 		)
-		(property "Value" "100nF/50V(10%)"
+		(property "Value" "100nF/50V"
 			(at 0 1.68 0)
 			(layer "F.Fab")
@@
 			)
 		)
-		(property "Value" "100nF/50V(10%)"
+		(property "Value" "100nF/50V"
 			(at 0 1.68 90)
 			(layer "F.Fab")
@@
 			)
 		)
-		(property "Value" "11k (1%)"
+		(property "Value" "11k"
 			(at 0 -1.65 90)
 			(layer "B.Fab")
@@
 			)
 		)
-		(property "Value" "3k (1%)"
+		(property "Value" "3k"
 			(at 0 -1.65 0)
 			(layer "B.Fab")
@@
 			)
 		)
-		(property "Value" "0.1uF/16V"
+		(property "Value" "100nF/16V"
 			(at 0 -1.43 0)
 			(layer "B.Fab")
@@
 			)
 		)
-		(property "Value" "2k2 (1%)"
+		(property "Value" "2k2"
 			(at 0 -1.65 90)
 			(layer "B.Fab")
@@
 			)
 		)
-		(property "Value" "1uF/16V(10%)"
+		(property "Value" "1uF/16V"
 			(at 0 -1.68 0)
 			(layer "B.Fab")
@@
 			)
 		)
-		(property "Value" "100nF/50V(10%)"
+		(property "Value" "100nF/50V"
 			(at 0 -1.68 90)
 			(layer "B.Fab")
@@
 			)
 		)
-		(property "Value" "5k1 (1%)"
+		(property "Value" "5k1"
 			(at 0 -1.65 0)
 			(layer "B.Fab")
@@
 			)
 		)
-		(property "Value" "1uF/16V(10%)"
+		(property "Value" "1uF/16V"
 			(at 0 -1.43 0)
 			(layer "B.Fab")
@@
 			)
 		)
-		(property "Value" "100nF/50V(10%)"
+		(property "Value" "100nF/50V"
 			(at 0 -1.68 90)
 			(layer "B.Fab")
@@
 			)
 		)
-		(property "Value" "100nF/50V(10%)"
+		(property "Value" "100nF/50V"
 			(at 0 -1.68 90)
 			(layer "B.Fab")
@@
 			)
 		)
-		(property "Value" "2k2 (1%)"
+		(property "Value" "2k2"
 			(at 0 -1.65 90)
 			(layer "B.Fab")
@@
 			)
 		)
-		(property "Value" "1uF/16V(10%)"
+		(property "Value" "1uF/16V"
 			(at 0 -1.43 90)
 			(layer "B.Fab")
@@
 			)
 		)
-		(property "Value" "LESD5D5.0CT1G"
+		(property "Value" "ESD5B5V0WT"
 			(at 0 -1.4 90)
 			(layer "B.Fab")
@@
 			)
 		)
-		(property "Value" "2k2 (1%)"
+		(property "Value" "2k2"
 			(at 0 -1.65 90)
 			(layer "B.Fab")
@@
 			)
 		)
-		(property "Value" "LESD5D5.0CT1G"
+		(property "Value" "ESD5B5V0WT"
 			(at 0 -1.4 0)
 			(layer "B.Fab")
@@
 			)
 		)
-		(property "Value" "5k1 (1%)"
+		(property "Value" "5k1"
 			(at 0 -1.65 0)
 			(layer "B.Fab")
