File: imu_rc_hand_unit/pcb/v1.1.0/imu_rc_hand_unit.kicad_sch (KiCad schematic)
At the start: 84 parts, among them J1 USB_C_Receptacle, J2 JST SH1.0, J3 USB_C_Receptacle_USB2.0_16P, Q1 AO3400A, Q2 AO3400A, Q3 AO3401A, Q4 AO3400A, Q5 AO3401A, Q6 BSS138, Q8 2N2907A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

Commit message: commit #36
added project report
few changes in imu rc car chassis for 3d printing
fixed some imu rc car pin outputs
major folder hierarchy refactor in pcb hand unit

imu rc hand unit v1.2.0:
changed footprint of MCP73831 to DFN-8
added 3V3 to VIO pin in CP2102N

new imu rc hand unit v2.0.0:
Changed to MCP73871
Removed BQ297
Removed a few components
only schematic is done
Parts:
- removed C16: 2n2F/16V, Capacitor_SMD:C_0805_2012Metric, symbol Device:C_Small
- removed C21, C23: 100nF/16V, Capacitor_SMD:C_0805_2012Metric, symbol Device:C_Small
- removed C22: 10nF/16V, Capacitor_SMD:C_0805_2012Metric, symbol Device:C_Small
- removed J1: USB_C_Receptacle, Library:USB_C_Receptacle_GCT_USB4110, symbol Connector:USB_C_Receptacle
- removed J3: USB_C_Receptacle_USB2.0_16P, symbol Connector:USB_C_Receptacle_USB2.0_16P
- removed Q9: 2N2907A, Package_TO_SOT_SMD:SOT-23, symbol Simulation_SPICE:NPN
- removed R52: 0, Resistor_SMD:R_1206_3216Metric, symbol Device:R_US
- removed U1: CP2102N, Package_DFN_QFN:QFN-24-1EP_4x4mm_P0.5mm_EP2.6x2.6mm, symbol Interface_USB:CP2102N-Axx-xQFN24
- removed U2: MCP73831, Package_DFN_QFN:QFN-20-1EP_4x4mm_P0.5mm_EP2.5x2.5mm, symbol Battery_Management:MCP73831-2-OT
- removed U7: MPU-6050, Sensor_Motion:InvenSense_QFN-24_4x4mm_P0.5mm, symbol Sensor_Motion:MPU-6050
- added C8: 100nF/50V, Capacitor_SMD:C_0805_2012Metric, symbol Device:C_Small
- added J1: USB_C_Receptacle_USB2.0_16P, Connector_USB:USB_C_Receptacle_GCT_USB4105-xx-A_16P_TopMnt_Horizontal, symbol Connector:USB_C_Receptacle_USB2.0_16P
- added Q7: BC817-25, Package_TO_SOT_SMD:SOT-23, symbol Simulation_SPICE:NPN
- added R19: 10k, Resistor_SMD:R_0805_2012Metric, symbol Device:R_US
- added U1: LSM6DSO, IMURCLibrary:LGA-14L_3x2.5mm_P0.5mm, symbol Sensor_Motion:LSM6DS3
- added U2: MCP73831-2-MC, Package_DFN_QFN:DFN-8-1EP_3x2mm_P0.5mm_EP1.7x1.4mm, symbol Battery_Management:MCP73831-2-MC
- added U6: CP2102N, Package_DFN_QFN:QFN-24-1EP_4x4mm_P0.5mm_EP2.6x2.6mm, symbol Interface_USB:CP2102N-Axx-xQFN24
- C12: value 100nF/50V(10%) -> 100nF/50V
- C13, C2, C4: value 1uF/16V(10%) -> 1uF/16V
- C14, C15, C17, C18, C19, C20: value 0.1uF/50V(10%) -> 100nF/50V
- C5: value 0.1uF/16V -> 100nF/16V
- D1, D2, D3: value LESD5D5.0CT1G -> ESD5B5V0WT
- D7: footprint MyLibrary:LED_D5.0mm-4_RKGB -> IMURCLibrary:LED_D5.0mm-4_RKGB
- J2: footprint Connector_JST:JST_SH_SM04B-SRSS-TB_1x04-1MP_P1.00mm_Horizontal -> IMURCLibrary:JST_SH_SM04B-SRSS-TB_1x04-1MP_P1.00mm_Horizontal
- Q1, Q2, Q4: value AO3400A -> IRLML6344TRPBF
- Q3, Q5: value AO3401A -> DMP3160L-7
- Q8: value 2N2907A -> BC817-25
- R13: value 6k -> 3k
- R14: value 22k -> 11k
- R24: value 10k -> 0; footprint Resistor_SMD:R_0805_2012Metric -> Resistor_SMD:R_1206_3216Metric
- R3: value 47k5 -> 22k1
- R31: value 150 -> 330
- R32: value 33 -> 68
- R33: value 10 -> 68
- R4: value 22k1 -> 47k5
Connections:
- net +3.3V: now also C8.1, U1.1 (SDO/SA0), U1.12 (CS), U1.2 (SDX), U1.3 (SCX), U1.5 (VDDIO), U1.8 (VDD), U6.5 (VIO), U6.6 (VDD), U6.7 (VREGIN)
- net +BATT: now also Q5.2 (S), U2.3 (V_{BAT}), U2.4 (V_{BAT}); no longer Q5.3 (D)
- net BATT_READ: now also U5.22 (GPIO14/TOUCH14/ADC2_CH3/FSPIWP/FSPIDQS/SUBSPIWP); no longer U5.34 (MTDI/GPIO41/CLK_OUT1)
- net BATT_READ_EN: now also U5.23 (GPIO21); no longer U5.35 (MTMS/GPIO42)
- net BOOT: now also R24.2
- net CHRG: now also U5.7 (GPIO7/TOUCH7/ADC1_CH6); no longer U5.33 (MTDO/GPIO40/CLK_OUT2)
- net CHRG_5V: now also U2.5 (STAT)
- net DTR: now also Q8.3 (E), R19.1, U6.23 (~{DTR}); no longer R22.1
- net GND: now also R4.1, C8.2, J1.A1 (GND), J1.A12 (GND), J1.B1 (GND), J1.B12 (GND), J1.S1 (SHIELD), U1.6 (GND), U1.7 (GND), U2.6 (V_{SS}), U6.2 (GND), U6.25 (GND); no longer R3.1
- net LED_BLUE: now also U5.4 (GPIO4/TOUCH4/ADC1_CH3); no longer U5.25 (GPIO48/SPICLK_N/SUBSPICLK_N_DIFF)
- net LED_GREEN: now also U5.5 (GPIO5/TOUCH5/ADC1_CH4); no longer U5.24 (GPIO47/SPICLK_P/SUBSPICLK_P_DIFF)
- net LED_RED: now also U5.6 (GPIO6/TOUCH6/ADC1_CH5); no longer U5.23 (GPIO21)
- net RTS: now also R22.1, Q7.3 (E), U6.19 (~{RTS}); no longer Q8.3 (E), R24.1
- net SCL: now also U1.13 (SCL)
- net SDA: now also U1.14 (SDA)
- net SW_DOWN: now also U5.11 (GPIO18/U1RXD/ADC2_CH7/CLK_OUT3); no longer U5.39 (GPIO1/TOUCH1/ADC1_CH0)
- net SW_FN: now also U5.8 (GPIO15/U0RTS/ADC2_CH4/XTAL_32K_P); no longer U5.26 (GPIO45)
- net SW_SLT: now also U5.10 (GPIO17/U1TXD/ADC2_CH6); no longer U5.38 (GPIO2/TOUCH2/ADC1_CH1)
- net SW_UP: now also U5.9 (GPIO16/U0CTS/ADC2_CH5/XTAL_32K_N); no longer U5.29 (SPIIO7/GPIO36/FSPICLK/SUBSPICLK)
- net U0RXD: now also U6.21 (TXD)
- net U0TXD: now also U6.20 (RXD)
- net VBUS: now also R3.2, U2.1 (V_{DD}), U2.2 (V_{DD}); no longer R4.2
- net at R7.1: now also U2.8 (PROG)
- net at R6.1: now also U6.15 (~{SUSPEND})
- net at R23.1: now also Q7.1 (C); no longer Q8.1 (C)
- net at D2.2 (A2): now also J1.A7 (D-), J1.B7 (D-), U6.4 (D-)
- net at D1.2 (A2), D4.2 (A): now also J1.A4 (VBUS), J1.A9 (VBUS), J1.B4 (VBUS), J1.B9 (VBUS)
- net at R2.2: now also J1.A5 (CC1)
- net at D3.2 (A2): now also J1.A6 (D+), J1.B6 (D+), U6.3 (D+)
- net at R1.2: now also J1.B5 (CC2)
- net at R5.1: now also U6.9 (~{RST})
- net at R13.1: now also Q5.3 (D); no longer Q5.2 (S)
- new net: C2.1, R3.1, R4.2, U6.8 (VBUS)
- new net: Q7.2 (B), R19.2
- new net: Q8.1 (C), R24.1
- no-connect marks 45 -> 35
Other:
- note added: "IC Buttons RTS/CTS"
- note added: "IMU"
- note added: "USB-C / UART"
- note added: "Voltage Regulator and Power Source Selector"
- note removed: "Buttons and power-up"
- note removed: "MPU-6050"
- note removed: "USB-C to UART"
- note removed: "Voltage Regulator w/ UPS"
- moved on the sheet: BOOT1, BT1, C1, C11, C12, C13, C14, C15, C17, C18, C19, C20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
