File: imu_rc_hand_unit/pcb/v2.0.0/imu_rc_hand_unit.kicad_sch (KiCad schematic)
At the start: 80 parts, among them J1 USB_C_Receptacle_USB2.0_16P, J2 JST SH1.0, Q1 IRLML6344TRPBF, Q2 IRLML6344TRPBF, Q3 DMP3160L-7, Q4 IRLML6344TRPBF, Q5 DMP3160L-7, Q6 BSS138, Q7 BC817-25, Q8 BC817-25, SW1 SW_SPDT, U1 LSM6DSO, U2 MCP73831, U3 BQ297xy, U4 AP2112K-3.3, U5 ESP32-S3-WROOM-1, U6 CP2102N

Commit message: commit #36
added project report
few changes in imu rc car chassis for 3d printing
fixed some imu rc car pin outputs
major folder hierarchy refactor in pcb hand unit

imu rc hand unit v1.2.0:
changed footprint of MCP73831 to DFN-8
added 3V3 to VIO pin in CP2102N

new imu rc hand unit v2.0.0:
Changed to MCP73871
Removed BQ297
Removed a few components
only schematic is done
Parts:
- removed C4: 1uF/16V(10%), Capacitor_SMD:C_0603_1608Metric, symbol Device:C_Small
- removed Q1, Q2: IRLML6344TRPBF, Package_TO_SOT_SMD:SOT-23, symbol Transistor_FET:AO3400A
- removed Q6: BSS138, Package_TO_SOT_SMD:SOT-23, symbol Transistor_FET:BSS138
- removed R15, R23, R24: 0, Resistor_SMD:R_1206_3216Metric, symbol Device:R_US
- removed R16, R17: 10k, Resistor_SMD:R_0805_2012Metric, symbol Device:R_US
- removed U2: MCP73831, Package_DFN_QFN:QFN-20-1EP_4x4mm_P0.5mm_EP2.5x2.5mm, symbol Battery_Management:MCP73831-2-OT
- removed U3: BQ297xy, Package_SON:WSON-6_1.5x1.5mm_P0.5mm, symbol Battery_Management:BQ297xy
- removed U5: ESP32-S3-WROOM-1, PCM_Espressif:ESP32-S3-WROOM-1, symbol PCM_Espressif:ESP32-S3-WROOM-1
- added C2: 10uF/16V, Capacitor_SMD:C_0805_2012Metric, symbol Device:C_Small
- added C6: 4u7F/16V, Capacitor_SMD:C_0805_2012Metric, symbol Device:C_Small
- added R11: 10k, Resistor_SMD:R_0805_2012Metric, symbol Device:R_US
- added U2: ESP32-S3-WROOM-2, PCM_Espressif:ESP32-S3-WROOM-2, symbol PCM_Espressif:ESP32-S3-WROOM-2
- added U7: MCP73871-2CC, Package_DFN_QFN:QFN-20-1EP_4x4mm_P0.5mm_EP2.5x2.5mm, symbol Battery_Management:MCP73871-2CC
- C10: renamed from C13; value 1uF/16V(10%) -> 1uF/16V
- C11: value 10uF/25V -> 10uF/16V
- C12: value 100nF/50V(10%) -> 100nF/50V
- C13: renamed from C17; value 100nF/50V(10%) -> 100nF/50V
- C14: renamed from C19; value 100nF/50V(10%) -> 100nF/50V
- C15: renamed from C18; value 100nF/50V(10%) -> 100nF/50V
- C16: renamed from C20; value 100nF/50V(10%) -> 100nF/50V
- C17: renamed from C15; value 100nF/50V(10%) -> 100nF/50V
- C18: renamed from C14; value 100nF/50V(10%) -> 100nF/50V
- C3: value 10uF/25V -> 10uF/16V; footprint Capacitor_SMD:C_0603_1608Metric -> Capacitor_SMD:C_0805_2012Metric
- C4: renamed from C2; value 1uF/16V(10%) -> 1uF/16V; footprint Capacitor_SMD:C_0603_1608Metric -> Capacitor_SMD:C_0805_2012Metric
- C5: value 0.1uF/16V -> 4u7F/16V; footprint Capacitor_SMD:C_0603_1608Metric -> Capacitor_SMD:C_0805_2012Metric
- C9: renamed from C8; value 100nF/50V(10%) -> 100nF/50V
- D1, D2: value LESD5D5.0CT1G -> ESD5B5V0WT
- R1, R2: value 5k1 (1%) -> 5k1
- R10: value 330 -> 10k
- R14: renamed from R13; value 3k (1%) -> 3k
- R15: renamed from R14; value 11k (1%) -> 11k
- R17: renamed from R20; value 2k2 (1%) -> 2k2
- R18: renamed from R21; value 2k2 (1%) -> 2k2
- R7: value 2k -> 1k
- R8: value 2k -> 20k
- R9: value 2k2 (1%) -> 10k
- renumbered SW_FN1 to BTN1, SW_SLT1 to BTN2, SW_UP1 to BTN3, SW_DOWN1 to BTN4, BOOT1 to BTN5, RESET1 to BTN6, C6 to C7, C7 to C8, Q3 to Q1, Q5 to Q2, Q4 to Q3, Q7 to Q4, Q8 to Q5, R11 to R12, R12 to R13, R18 to R16, R25 to R19, R29 to R20, R28 to R21, R30 to R22, R27 to R23, R26 to R24, R19 to R25, R22 to R26, R6 to R5, R5 to R6
Connections:
- net CHRG_5V is gone; now on net GND: R8.2
- net +3.3V: now also R10.1, R9.1, U6.5 (VIO), R11.1, U2.2 (3V3)
- net +BATT: now also C6.1, U7.1 (OUT), U7.20 (OUT); no longer R10.2, SW1.3 (C)
- net BATT_READ: now also U2.22 (GPIO14/TOUCH14/ADC2_CH3/FSPIWP/FSPIDQS/SUBSPIWP)
- net BATT_READ_EN: now also U2.23 (GPIO21)
- net BOOT: now also Q5.1 (C), U2.27 (GPIO0/BOOT)
- net CHIP_PU: now also Q4.1 (C), U2.3 (EN)
- net GND: now also BT1.2 (-), C5.2, C2.2, C6.2, U2.1 (GND), U2.40 (GND), U2.41 (GND), U7.10 (V_{SS}), U7.11 (V_{SS}), U7.21 (V_{SS}), U7.3 (SEL); no longer R9.1
- net LED_BLUE: now also U2.4 (GPIO4/TOUCH4/ADC1_CH3)
- net LED_GREEN: now also U2.5 (GPIO5/TOUCH5/ADC1_CH4)
- net LED_RED: now also U2.6 (GPIO6/TOUCH6/ADC1_CH5)
- net SCL: now also U2.17 (GPIO9/TOUCH9/ADC1_CH8/FSPIHD/SUBSPIHD)
- net SDA: now also U2.12 (GPIO8/TOUCH8/ADC1_CH7/SUBSPICS1)
- net U0RXD: now also U2.36 (U0RXD/GPIO44/CLK_OUT2)
- net U0TXD: now also U2.37 (U0TXD/GPIO43/CLK_OUT1)
- net VBUS: now also C2.1, U7.17 (CE), U7.18 (IN), U7.19 (IN), U7.2 (VPCC), U7.4 (PROG2), U7.9 (~{TE}); no longer R8.1
- net at R7.1: now also U7.13 (PROG1)
- net at C5.1: now also SW1.1 (A), U7.14 (V_{BAT}), U7.15 (V_{BAT}), U7.16 (V_{BAT_SENSE}); no longer R10.1
- net PG: now reaches R9.2
- net PG: now also U7.6 (~{PG})
- net SW_DOWN renamed SW_4
- net SW_4: now also U2.11 (GPIO18/U1RXD/ADC2_CH7/CLK_OUT3)
- net SW_FN renamed SW_1
- net SW_1: now also U2.8 (GPIO15/U0RTS/ADC2_CH4/XTAL_32K_P)
- net SW_SLT renamed SW_3
- net SW_3: now also U2.10 (GPIO17/U1TXD/ADC2_CH6)
- net SW_UP renamed SW_2
- net SW_2: now also U2.9 (GPIO16/U0CTS/ADC2_CH5/XTAL_32K_N)
- new net: R8.1, U7.12 (PROG3)
- new net STAT1: R10.2, U7.8 (STAT1/~{LBO})
- new net STAT2: R11.2, U7.7 (STAT2)
- no-connect marks 36 -> 33
Other:
- note added: "Battery Charger and Reader"
- note added: "FN Buttons"
- note added: "USB-C and USB/UART Converter"
- note removed: "Battery Charger w/ 1S BMS"
- note removed: "Battery Reader"
- note removed: "Function Buttons"
- note removed: "IC Buttons RTS/CTS"
- note removed: "USB-C / UART"
- title: IMU-RC Hand Unit -> IMU-RC Hand Unit V2
- moved on the sheet: BT1, BTN2, BTN3, BTN4, BTN5, BTN6, C10, C11, C12, C14, C15, C16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
